File: watch-pcb/watch.kicad_pcb (KiCad board)
At the start: 2 copper layers, 11 parts, among them J1 Conn_01x02, J2 Conn_01x08, J3 Conn_01x02_Female, U1 NCP161, U2 ATmega328-A, U3 RFM69HCW, U4 PCF85263ATT

Commit message: working on layout
Parts:
- C1, C2, R1, R2, U1, U2, U4: moved to B.Cu
- J2: footprint Connector_PinHeader_2.54mm:PinHeader_1x08_P2.54mm_Vertical -> E-Ink:Waveshare_1.54
- U3: footprint Package_DIP:SMDIP-16_W7.62mm -> RFM69:RFM69HCW
- moved J2 117.2 mm to (168.0, 102.0)
- moved U2 106.9 mm to (155.0, 118.0), turned to -90 degrees
- moved R1 102.8 mm to (155.1, 128.0), turned to 180 degrees
- moved R2 100.0 mm to (147.1, 128.0), turned to 180 degrees
- moved U4 82.6 mm to (143.0, 118.0), turned to -90 degrees
- moved C1 77.5 mm to (138.0, 95.5), turned to -90 degrees
- moved U1 64.3 mm to (132.9, 95.5), turned to 180 degrees
- moved C2 59.6 mm to (127.8, 95.5), turned to -90 degrees
- moved U3 54.1 mm to (144.0, 93.5)
- moved J1 46.4 mm to (116.8, 81.3)
- moved J3 37.2 mm to (106.7, 81.3)
Other:
- board outline added: 48 x 33 mm

Commit message: layout in progress
Parts:
- added C3: 0.1uF, Capacitor_SMD:C_0603_1608Metric_Pad1.08x0.95mm_HandSolder, F.Cu at (109.2, 109.2)
- added C4: 0.1uF, Capacitor_SMD:C_0603_1608Metric_Pad1.08x0.95mm_HandSolder, F.Cu at (109.2, 111.7)
- added C5: 0.1uF, Capacitor_SMD:C_0603_1608Metric_Pad1.08x0.95mm_HandSolder, F.Cu at (90.8, 115.6)
- added J4: Conn_01x08, Connector_PinHeader_2.00mm:PinHeader_2x04_P2.00mm_Vertical, B.Cu at (136.0, 88.0)
- added N1: Battery, Battery:LiPo-100mAh, F.Cu at (125.5, 125.0)
- added R3: 10k, Resistor_SMD:R_0603_1608Metric_Pad0.98x0.95mm_HandSolder, F.Cu at (104.9, 114.2)
- added R4: 4.7k, Resistor_SMD:R_0603_1608Metric_Pad0.98x0.95mm_HandSolder, F.Cu at (104.9, 111.7)
- added R5: 4.7k, Resistor_SMD:R_0603_1608Metric_Pad0.98x0.95mm_HandSolder, F.Cu at (104.9, 109.2)
- added SW1: EVQ-P4MB3K, TinySwitch:EVQ-P4, F.Cu at (122.6, 108.5)
- added SW2: EVQ-P4MB3K, TinySwitch:EVQ-P4, F.Cu at (122.6, 116.5)
- added SW3: EVQ-P4MB3K, TinySwitch:EVQ-P4, F.Cu at (122.6, 100.5)
- added SW4: EVQ-P4MB3K, TinySwitch:EVQ-P4, F.Cu at (176.9, 95.5)
- J1, J3: footprint Connector_PinHeader_2.54mm:PinHeader_1x02_P2.54mm_Vertical -> Connector_PinSocket_2.00mm:PinSocket_1x02_P2.00mm_Vertical
- moved J3 62.4 mm to (163.5, 107.0), turned to 180 degrees
- moved J1 27.0 mm to (131.5, 104.0), turned to 90 degrees
- moved U2 1.50 mm to (156.5, 118.0)
- moved U4 1.50 mm to (144.5, 118.0)
Connections:
- net /eCLK renamed /SCK
- net /eDIN renamed /MOSI
- net Net-(U2-Pad14) renamed /RF_CS
- net Net-(U2-Pad16) renamed /MISO
- net Net-(U2-Pad27) renamed /SCL
- net Net-(U2-Pad28) renamed /SDA
- U2 pad 1: unconnected-(U2-Pad1) -> Net-(SW4-Pad1)
- U2 pad 24: unconnected-(U2-Pad24) -> Net-(SW1-Pad1)
- U2 pad 25: unconnected-(U2-Pad25) -> Net-(SW2-Pad1)
- U2 pad 29: unconnected-(U2-Pad29) -> /nRESET
- U2 pad 30: unconnected-(U2-Pad30) -> /RXD
- U2 pad 31: unconnected-(U2-Pad31) -> /TXD
- U2 pad 32: Net-(U2-Pad32) -> Net-(SW3-Pad1)
- U2 pad 9: unconnected-(U2-Pad9) -> Net-(U2-Pad9)
- U3 pad 14: Net-(U2-Pad32) -> Net-(U2-Pad9)
Other:
- outline, holes or cut-outs redrawn

Commit message: working on layout
Parts:
- C1, C2: footprint Capacitor_SMD:C_0603_1608Metric_Pad1.08x0.95mm_HandSolder -> Capacitor_SMD:C_0603_1608Metric; moved to F.Cu
- C3, C4, C5: footprint Capacitor_SMD:C_0603_1608Metric_Pad1.08x0.95mm_HandSolder -> Capacitor_SMD:C_0603_1608Metric
- J1, J3: moved to B.Cu
- J4: footprint Connector_PinHeader_2.00mm:PinHeader_2x04_P2.00mm_Vertical -> Connector_PinSocket_2.00mm:PinSocket_2x04_P2.00mm_Vertical_SMD
- R1, R2: footprint Resistor_SMD:R_0603_1608Metric_Pad0.98x0.95mm_HandSolder -> Resistor_SMD:R_0603_1608Metric; moved to F.Cu
- R3, R4, R5: footprint Resistor_SMD:R_0603_1608Metric_Pad0.98x0.95mm_HandSolder -> Resistor_SMD:R_0603_1608Metric
- U1: moved to F.Cu
- moved C5 57.2 mm to (148.0, 114.1), turned to 90 degrees
- moved C4 55.2 mm to (163.0, 99.5), turned to -90 degrees
- moved R5 49.7 mm to (153.8, 118.0), turned to 90 degrees
- moved SW1 49.6 mm to (171.5, 116.2), turned to 90 degrees
- moved C3 48.3 mm to (157.2, 114.5), turned to 90 degrees
- moved R4 46.6 mm to (151.0, 118.0), turned to 90 degrees
- moved R3 43.3 mm to (148.0, 117.9), turned to 90 degrees
- moved R2 13.7 mm to (156.5, 118.0), turned to 90 degrees
- moved SW4 12.5 mm to (165.4, 100.5)
- moved J4 11.6 mm to (134.5, 99.5)
- moved C1 11.0 mm to (127.4, 98.5)
- moved R1 10.7 mm to (159.0, 118.0), turned to -90 degrees
- moved C2 10.2 mm to (137.6, 98.5)
- moved J1 6.00 mm to (125.5, 104.0), turned to 0 degrees
- moved U1 3.03 mm to (132.5, 98.5), turned to 0 degrees
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Other:
- outline, holes or cut-outs redrawn

Commit message: Update 3D
Parts:
- removed SW1: EVQ-P4MB3K, TinySwitch:EVQ-P4
Changed lines of the file:
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@@
-    )
-  )
-  (footprint "TinySwitch:EVQ-P4" (layer "F.Cu")
-    (at 171.5 116.25 90)
-    (property "CatNo" "P15507CT-ND")
-    (property "Sheetfile" "File: watch.kicad_sch")
-    (property "Sheetname" "")
-    (attr smd)
-    (fp_text reference "SW1" (at 5 0.75 unlocked) (layer "F.SilkS")
-      (effects (font (size 1 1) (thickness 0.15)))
-    )
-    (fp_text value "EVQ-P4MB3K" (at 5.08 -2.54 90 unlocked) (layer "F.Fab")
-      (effects (font (size 1 1) (thickness 0.15)))
-    )
-    (fp_text user "${REFERENCE}" (at 5.08 -5.08 90 unlocked) (layer "F.Fab")
-      (effects (font (size 1 1) (thickness 0.15)))
-    )
-    (fp_line (start 2.55 2.6) (end 3.1 2.6) (layer "F.SilkS") (width 0.12))
-    (fp_line (start -2.55 2.6) (end -2.55 0.825) (layer "F.SilkS") (width 0.12))
-    (fp_line (start 2.55 2.6) (end 2.55 0.825) (layer "F.SilkS") (width 0.12))
-    (fp_line (start -2.55 2.6) (end -3.1 2.6) (layer "F.SilkS") (width 0.12))
-    (fp_line (start -2.55 0.825) (end 2.55 0.825) (layer "F.SilkS") (width 0.12))
-    (fp_rect (start -3.5 2.6) (end 3.6 -0.5) (layer "F.CrtYd") (width 0.05) (fill none))
-    (pad "1" smd rect (at -2.275 0 90) (size 1.45 1.05) (layers "F.Cu" "F.Paste" "F.Mask")
-      (net 25 "Net-(SW1-Pad1)") (pinfunction "1") (pintype "passive"))
-    (pad "2" smd rect (at 2.275 0 90) (size 1.45 1.05) (layers "F.Cu" "F.Paste" "F.Mask")
-      (net 2 "GND") (pinfunction "2") (pintype "passive"))
-    (pad "3" smd rect (at -3.2 1.75 90) (size 0.6 0.8) (layers "F.Cu" "F.Paste" "F.Mask"))
-    (pad "4" smd rect (at 3.2 1.75 90) (size 0.6 0.8) (layers "F.Cu" "F.Paste" "F.Mask"))
-    (model "/home/hazen/work/watch/3D/EVQP4-HB3B_KB3Q_MB3K.STEP"
-      (offset (xyz 0 -2.7 -0.5))
-      (scale (xyz 1 1 1))
-      (rotate (xyz 90 0 180))
     )
   )
@@
       (effects (font (size 1 1) (thickness 0.15)))
     )
-    (fp_line (start 0 23.5) (end 0 15.5) (layer "F.SilkS") (width 0.12))
+    (fp_line (start -48 -9.5) (end -48 23.5) (layer "F.SilkS") (width 0.12))
+    (fp_line (start 0 -9.5) (end 0 -1.5) (layer "F.SilkS") (width 0.12))
     (fp_line (start 0 -9.5) (end -48 -9.5) (layer "F.SilkS") (width 0.12))
     (fp_line (start -48 23.5) (end 0 23.5) (layer "F.SilkS") (width 0.12))
-    (fp_line (start 0 -9.5) (end 0 -1.5) (layer "F.SilkS") (width 0.12))
-    (fp_line (start -48 -9.5) (end -48 23.5) (layer "F.SilkS") (width 0.12))
+    (fp_line (start 0 23.5) (end 0 15.5) (layer "F.SilkS") (width 0.12))
+    (pad "" np_thru_hole circle (at -2.5 -7) (size 2.7 2.7) (drill 2.7) (layers F&B.Cu *.Mask))
+    (pad "" np_thru_hole circle (at -45.5 20.5) (size 2.7 2.7) (drill 2.7) (layers F&B.Cu *.Mask))
     (pad "" np_thru_hole circle (at -45.5 -7) (size 2.7 2.7) (drill 2.7) (layers F&B.Cu *.Mask))
-    (pad "" np_thru_hole circle (at -45.5 20.5) (size 2.7 2.7) (drill 2.7) (layers F&B.Cu *.Mask))
-    (pad "" np_thru_hole circle (at -2.5 -7) (size 2.7 2.7) (drill 2.7) (layers F&B.Cu *.Mask))
     (pad "" np_thru_hole circle (at -2.5 21) (size 2.7 2.7) (drill 2.7) (layers F&B.Cu *.Mask))
     (pad "1" smd roundrect (at -1.5 3.5) (size 2.286 1.524) (layers "B.Cu" "B.Paste" "B.Mask") (roundrect_rratio 0.25)
@@
     (pad "8" smd roundrect (at -1.5 17.5) (size 2.286 1.524) (layers "B.Cu" "B.Paste" "B.Mask") (roundrect_rratio 0.25)
       (net 3 "+3.3V") (pinfunction "Pin_8") (pintype "passive"))
+    (model "/home/hazen/work/watch/3D/watch-Matrix_Union002.step"
+      (offset (xyz 0 -23.6 6))
+      (scale (xyz 1 1 1))
+      (rotate (xyz 0 0 -90))
+    )
   )
   (footprint "Resistor_SMD:R_0603_1608Metric" (layer "F.Cu")

Commit message: as built PCB rev 1.0
Parts:
- added D1: LED, LED_SMD:LED_0603_1608Metric_Pad1.05x0.95mm_HandSolder, B.Cu at (146.5, 123.4)
- added D2: LED, LED_SMD:LED_0603_1608Metric_Pad1.05x0.95mm_HandSolder, B.Cu at (144.2, 123.4)
- added R6: 330, Resistor_SMD:R_0603_1608Metric, F.Cu at (146.6, 123.4)
- added R7: 330, Resistor_SMD:R_0603_1608Metric, F.Cu at (144.2, 123.4)
- moved U3 1.50 mm to (144.0, 93.5)
- moved J2 0.05 mm to (167.9, 102.0)
- turned R1 to 90 degrees
Connections:
- U2 pad 7: unconnected-(U2-Pad7) -> /LED1
- U2 pad 8: unconnected-(U2-Pad8) -> /LED2
Routing:
- net Net-(C1-Pad1): track 0.00 -> 76.1 mm, vias 0 -> 2
- net /SCK: track 0.00 -> 70.7 mm, vias 0 -> 7
- net /MISO: track 0.00 -> 60.6 mm, vias 0 -> 3
- net /MOSI: track 0.00 -> 58.8 mm, vias 0 -> 6
- net Net-(SW2-Pad1): track 0.00 -> 52.8 mm, vias 0 -> 5
- net Net-(SW3-Pad1): track 0.00 -> 50.1 mm, vias 0 -> 3
- net /RXD: track 0.00 -> 41.7 mm, vias 0 -> 4
- net /nRESET: track 0.00 -> 40.4 mm, vias 0 -> 4
- net /RF_CS: track 0.00 -> 39.1 mm, vias 0 -> 3
- net Net-(U2-Pad23): track 0.00 -> 38.1 mm, vias 0 -> 3
- net GND: track 0.00 -> 37.8 mm, vias 0 -> 17
- net /LED2: track 0.00 -> 32.4 mm, vias 0 -> 3
- net +3.3V: track 0.00 -> 31.6 mm, vias 0 -> 13
- net /TXD: track 0.00 -> 31.1 mm, vias 0 -> 2
- net /LED1: track 0.00 -> 25.3 mm, vias 0 -> 1
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- added copper zone on In2.Cu, net +3.3V
- added copper zone on In1.Cu, net GND
Other:
- outline, holes or cut-outs redrawn
- copper layers 2 -> 4
- board text added: "+"
- board text added: "-"
- board text added: "1"
- board text added: "ANT"
- board text added: "BAT"
- board text added: "PROG/TEST"
- board text added: "UPCO Watch V1.0"

Commit message: readme
Parts:
- J2: footprint E-Ink:Waveshare_1.54 -> E-Ink:Waveshare_1.54_no3D
Changed lines of the file:
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@@
     )
   )
-  (footprint "E-Ink:Waveshare_1.54" (layer "F.Cu")
+  (footprint "E-Ink:Waveshare_1.54_no3D" (layer "F.Cu")
     (at 167.905 102)
     (property "Sheetfile" "watch.kicad_sch")
     (property "Sheetname" "")
     (attr smd)
-    (fp_text reference "J2" (at -0.905 19.25 unlocked) (layer "F.SilkS")
+    (fp_text reference "J2" (at -5 -11 unlocked) (layer "F.SilkS")
       (effects (font (size 1 1) (thickness 0.15)))
     )
@@
       (effects (font (size 1 1) (thickness 0.15)))
     )
-    (fp_line (start 0 23.5) (end 0 15.5) (layer "F.SilkS") (width 0.12))
-    (fp_line (start -48 23.5) (end 0 23.5) (layer "F.SilkS") (width 0.12))
     (fp_line (start 0 -9.5) (end -48 -9.5) (layer "F.SilkS") (width 0.12))
     (fp_line (start -48 -9.5) (end -48 23.5) (layer "F.SilkS") (width 0.12))
+    (fp_line (start -48 23.5) (end 0 23.5) (layer "F.SilkS") (width 0.12))
     (fp_line (start 0 -9.5) (end 0 -1.5) (layer "F.SilkS") (width 0.12))
+    (fp_line (start 0 23.5) (end 0 15.5) (layer "F.SilkS") (width 0.12))
     (pad "" np_thru_hole circle (at -2.5 -7) (size 2.7 2.7) (drill 2.7) (layers F&B.Cu *.Mask))
+    (pad "" np_thru_hole circle (at -2.5 21) (size 2.7 2.7) (drill 2.7) (layers F&B.Cu *.Mask))
+    (pad "" np_thru_hole circle (at -45.5 20.5) (size 2.7 2.7) (drill 2.7) (layers F&B.Cu *.Mask))
     (pad "" np_thru_hole circle (at -45.5 -7) (size 2.7 2.7) (drill 2.7) (layers F&B.Cu *.Mask))
-    (pad "" np_thru_hole circle (at -45.5 20.5) (size 2.7 2.7) (drill 2.7) (layers F&B.Cu *.Mask))
-    (pad "" np_thru_hole circle (at -2.5 21) (size 2.7 2.7) (drill 2.7) (layers F&B.Cu *.Mask))
     (pad "1" smd roundrect (at -1.5 3.5) (size 2.286 1.524) (layers "B.Cu" "B.Paste" "B.Mask") (roundrect_rratio 0.25)
       (net 4 "/eBUSY") (pinfunction "Pin_1") (pintype "passive"))
@@
     (pad "8" smd roundrect (at -1.5 17.5) (size 2.286 1.524) (layers "B.Cu" "B.Paste" "B.Mask") (roundrect_rratio 0.25)
       (net 3 "+3.3V") (pinfunction "Pin_8") (pintype "passive"))
-    (model "/home/hazen/work/watch/3D/watch-Matrix_Union002.step"
-      (offset (xyz 0 -23.6 6))
-      (scale (xyz 1 1 1))
-      (rotate (xyz 0 0 -90))
-    )
   )
   (footprint "Capacitor_SMD:C_0603_1608Metric" (layer "F.Cu")
