File: watch-pcb/watch.kicad_sch (KiCad schematic)
At the start: 1 part

Commit message: working on PCB
Parts:
- removed A?: Arduino_UNO_R3, Module:Arduino_UNO_R3, symbol MCU_Module:Arduino_UNO_R3
- added C1, C2: 1uF, Capacitor_SMD:C_0603_1608Metric_Pad1.08x0.95mm_HandSolder, symbol Device:C_Small
- added J1: Conn_01x02, Connector_PinHeader_2.54mm:PinHeader_1x02_P2.54mm_Vertical, symbol Connector_Generic:Conn_01x02
- added J2: Conn_01x08, Connector_PinHeader_2.54mm:PinHeader_1x08_P2.54mm_Vertical, symbol Connector_Generic:Conn_01x08
- added J3: Conn_01x02_Female, Connector_PinHeader_2.54mm:PinHeader_1x02_P2.54mm_Vertical, symbol Connector:Conn_01x02_Female
- added R1, R2: 10k, Resistor_SMD:R_0603_1608Metric_Pad0.98x0.95mm_HandSolder, symbol Device:R_US
- added U1: NCP161, Package_TO_SOT_SMD:SOT-23-5, symbol Regulator_Linear:LP2985-1.8
- added U2: ATmega328-A, Package_QFP:TQFP-32_7x7mm_P0.8mm, symbol MCU_Microchip_ATmega:ATmega328-A
- added U3: RFM69HCW, Package_DIP:SMDIP-16_W7.62mm, symbol RF_Module:RFM69HCW
- added U4: PCF85263ATT, Package_SO:TSSOP-8_3x3mm_P0.65mm, symbol Timer_RTC:PCF85263ATT
Connections:
- new net: C1.1, J1.1 (Pin_1), R1.1, U1.1 (VIN), U1.3 (ON/~{OFF})
- new net: R1.2, R2.1, U2.19 (ADC6)
- new net: J3.1 (Pin_1), U3.9 (ANT)
- new net: U2.28 (PC5), U4.5 (SDA)
- new net: U2.27 (PC4), U4.6 (SCL)
- new net: U2.26 (PC3), U4.7 (~{INTA})
- new net: U2.14 (PB2), U3.5 (NSS)
- new net: U2.16 (PB4), U3.2 (MISO)
- new net: U2.23 (PC0), U3.6 (RESET)
- new net: U2.32 (PD2), U3.14 (DIO0)
- new net +3.3V: C2.1, J2.8 (Pin_8), U1.5 (VOUT), U2.18 (AVCC), U2.20 (AREF), U2.4 (VCC), U2.6 (VCC), U3.13 (3.3V), U4.3 (VBAT), U4.8 (VDD)
- new net GND: C1.2, C2.2, J1.2 (Pin_2), J2.7 (Pin_7), J3.2 (Pin_2), R2.2, U1.2 (GND), U2.21 (GND), U2.3 (GND), U2.5 (GND), U3.1 (GND), U3.10 (GND), U3.8 (GND), U4.4 (VSS)
- new net eBUSY: J2.1 (Pin_1), U2.11 (PD7)
- new net eCLK: J2.5 (Pin_5), U2.17 (PB5), U3.4 (SCK)
- new net eCS: J2.4 (Pin_4), U2.10 (PD6)
- new net eDC: J2.3 (Pin_3), U2.13 (PB1)
- new net eDIN: J2.6 (Pin_6), U2.15 (PB3), U3.3 (MOSI)
- new net eRST: J2.2 (Pin_2), U2.12 (PB0)
- no-connect marks 0 -> 1
Other:
- note added: "915MHz ISM Transceiver"
- note added: "A"
- note added: "ATMega328 CPU (should really be e.g. ATMega1281 but supply chain...)"
- note added: "Battery"
- note added: "Real-time clock"
- note added: "Smart Watch"
- note added: "UPCO GRAPHICS SYSTEMS"
- note added: "Waveshare e-Ink"

Commit message: working on layout
Parts:
- added J4: Conn_01x08, symbol Connector_Generic:Conn_01x08
- added R3: 10k, Resistor_SMD:R_0603_1608Metric_Pad0.98x0.95mm_HandSolder, symbol Device:R_US
- added R4, R5: 4.7k, Resistor_SMD:R_0603_1608Metric_Pad0.98x0.95mm_HandSolder, symbol Device:R_US
- added SW1, SW2, SW3, SW4: EVQ-P4MB3K, symbol Switch:SW_Push
- J2: footprint Connector_PinHeader_2.54mm:PinHeader_1x08_P2.54mm_Vertical -> E-Ink:Waveshare_1.54
- U3: footprint Package_DIP:SMDIP-16_W7.62mm -> RFM69:RFM69HCW
Connections:
- net +3.3V: now also J4.1 (Pin_1), R3.1, R4.1, R5.1
- net GND: now also J4.8 (Pin_8), SW1.2, SW2.2, SW3.2, SW4.2
- net SDA: now reaches U2.28 (PC5), U4.5 (SDA)
- net SDA: now also R5.2
- net SCL: now reaches U2.27 (PC4), U4.6 (SCL)
- net SCL: now also R4.2
- net at U2.1 (PD3): now also SW4.1
- net RF_CS: now reaches U2.14 (PB2), U3.5 (NSS)
- net MISO: now reaches U2.16 (PB4), U3.2 (MISO)
- net MISO: now also J4.3 (Pin_3)
- net at U2.24 (PC1): now also SW1.1
- net at U2.25 (PC2): now also SW2.1
- net nRESET: now reaches U2.29 (~{RESET}/PC6)
- net nRESET: now also J4.5 (Pin_5), R3.2
- net RXD: now reaches U2.30 (PD0)
- net RXD: now also J4.7 (Pin_7)
- net TXD: now reaches U2.31 (PD1)
- net TXD: now also J4.6 (Pin_6)
- net at U2.32 (PD2): now also SW3.1; no longer U3.14 (DIO0)
- net at U2.9 (PD5): now also U3.14 (DIO0)
- net eCLK renamed SCK
- net SCK: now also J4.4 (Pin_4)
- net eDIN renamed MOSI
- net MOSI: now also J4.2 (Pin_2)
Other:
- note added: ""Service" connector"
- note added: "UART, AVR progr"

Commit message: layout in progress
Parts:
- added C3, C4, C5: 0.1uF, Capacitor_SMD:C_0603_1608Metric_Pad1.08x0.95mm_HandSolder, symbol Device:C_Small
- added N1: Battery, Battery:LiPo-100mAh, symbol Mechanical:Housing
- J1, J3: footprint Connector_PinHeader_2.54mm:PinHeader_1x02_P2.54mm_Vertical -> Connector_PinSocket_2.00mm:PinSocket_1x02_P2.00mm_Vertical
- J4: footprint (none) -> Connector_PinHeader_2.00mm:PinHeader_2x04_P2.00mm_Vertical
- SW1, SW2, SW3, SW4: footprint (none) -> TinySwitch:EVQ-P4
Connections:
- net +3.3V: now also C3.1, C4.1, C5.1
- net GND: now also C3.2, C4.2, C5.2

Commit message: working on layout
Parts:
- C1, C2, C3, C4, C5: footprint Capacitor_SMD:C_0603_1608Metric_Pad1.08x0.95mm_HandSolder -> Capacitor_SMD:C_0603_1608Metric
- J4: footprint Connector_PinHeader_2.00mm:PinHeader_2x04_P2.00mm_Vertical -> Connector_PinSocket_2.00mm:PinSocket_2x04_P2.00mm_Vertical_SMD
- R1, R2, R3, R4, R5: footprint Resistor_SMD:R_0603_1608Metric_Pad0.98x0.95mm_HandSolder -> Resistor_SMD:R_0603_1608Metric
Changed lines of the file:
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@@
       (effects (font (size 1.27 1.27)) (justify left))
     )
-    (property "Footprint" "Capacitor_SMD:C_0603_1608Metric_Pad1.08x0.95mm_HandSolder" (id 2) (at 48.895 45.72 0)
+    (property "Footprint" "Capacitor_SMD:C_0603_1608Metric" (id 2) (at 48.895 45.72 0)
       (effects (font (size 1.27 1.27)) hide)
     )
@@
       (effects (font (size 1.27 1.27)) (justify left))
     )
-    (property "Footprint" "Resistor_SMD:R_0603_1608Metric_Pad0.98x0.95mm_HandSolder" (id 2) (at 46.736 96.139 90)
+    (property "Footprint" "Resistor_SMD:R_0603_1608Metric" (id 2) (at 46.736 96.139 90)
       (effects (font (size 1.27 1.27)) hide)
     )
@@
       (effects (font (size 1.27 1.27)) (justify left))
     )
-    (property "Footprint" "Capacitor_SMD:C_0603_1608Metric_Pad1.08x0.95mm_HandSolder" (id 2) (at 193.04 106.68 0)
+    (property "Footprint" "Capacitor_SMD:C_0603_1608Metric" (id 2) (at 193.04 106.68 0)
       (effects (font (size 1.27 1.27)) hide)
     )
@@
       (effects (font (size 1.27 1.27)) (justify left))
     )
-    (property "Footprint" "Capacitor_SMD:C_0603_1608Metric_Pad1.08x0.95mm_HandSolder" (id 2) (at 81.915 45.72 0)
+    (property "Footprint" "Capacitor_SMD:C_0603_1608Metric" (id 2) (at 81.915 45.72 0)
       (effects (font (size 1.27 1.27)) hide)
     )
@@
       (effects (font (size 1.27 1.27)) (justify left))
     )
-    (property "Footprint" "Resistor_SMD:R_0603_1608Metric_Pad0.98x0.95mm_HandSolder" (id 2) (at 46.736 84.709 90)
+    (property "Footprint" "Resistor_SMD:R_0603_1608Metric" (id 2) (at 46.736 84.709 90)
       (effects (font (size 1.27 1.27)) hide)
     )
@@
       (effects (font (size 1.27 1.27)) (justify left))
     )
-    (property "Footprint" "Resistor_SMD:R_0603_1608Metric_Pad0.98x0.95mm_HandSolder" (id 2) (at 139.446 85.979 90)
+    (property "Footprint" "Resistor_SMD:R_0603_1608Metric" (id 2) (at 139.446 85.979 90)
       (effects (font (size 1.27 1.27)) hide)
     )
@@
       (effects (font (size 1.27 1.27)) (justify left))
     )
-    (property "Footprint" "Resistor_SMD:R_0603_1608Metric_Pad0.98x0.95mm_HandSolder" (id 2) (at 131.191 85.979 90)
+    (property "Footprint" "Resistor_SMD:R_0603_1608Metric" (id 2) (at 131.191 85.979 90)
       (effects (font (size 1.27 1.27)) hide)
     )
@@
       (effects (font (size 1.27 1.27)) (justify left))
     )
-    (property "Footprint" "Capacitor_SMD:C_0603_1608Metric_Pad1.08x0.95mm_HandSolder" (id 2) (at 97.79 66.04 0)
+    (property "Footprint" "Capacitor_SMD:C_0603_1608Metric" (id 2) (at 97.79 66.04 0)
       (effects (font (size 1.27 1.27)) hide)
     )
@@
     (property "Reference" "J4" (id 0) (at 23.495 146.05 0))
     (property "Value" "Conn_01x08" (id 1) (at 23.495 148.59 0))
-    (property "Footprint" "Connector_PinHeader_2.00mm:PinHeader_2x04_P2.00mm_Vertical" (id 2) (at 23.495 160.02 0)
+    (property "Footprint" "Connector_PinSocket_2.00mm:PinSocket_2x04_P2.00mm_Vertical_SMD" (id 2) (at 23.495 160.02 0)
       (effects (font (size 1.27 1.27)) hide)
     )
@@
       (effects (font (size 1.27 1.27)) (justify left))
     )
-    (property "Footprint" "Resistor_SMD:R_0603_1608Metric_Pad0.98x0.95mm_HandSolder" (id 2) (at 48.641 159.004 90)
+    (property "Footprint" "Resistor_SMD:R_0603_1608Metric" (id 2) (at 48.641 159.004 90)
       (effects (font (size 1.27 1.27)) hide)
     )
@@
       (effects (font (size 1.27 1.27)) (justify left))
     )
-    (property "Footprint" "Capacitor_SMD:C_0603_1608Metric_Pad1.08x0.95mm_HandSolder" (id 2) (at 135.89 33.02 0)
+    (property "Footprint" "Capacitor_SMD:C_0603_1608Metric" (id 2) (at 135.89 33.02 0)
       (effects (font (size 1.27 1.27)) hide)
     )
@@
     )
     (path "/05790f91-be61-4992-b5ba-7c0843162953"
-      (reference "C1") (unit 1) (value "1uF") (footprint "Capacitor_SMD:C_0603_1608Metric_Pad1.08x0.95mm_HandSolder")
+      (reference "C1") (unit 1) (value "1uF") (footprint "Capacitor_SMD:C_0603_1608Metric")
     )
     (path "/28a43f09-b358-4d07-aa48-59c5e610324f"
-      (reference "C2") (unit 1) (value "1uF") (footprint "Capacitor_SMD:C_0603_1608Metric_Pad1.08x0.95mm_HandSolder")
+      (reference "C2") (unit 1) (value "1uF") (footprint "Capacitor_SMD:C_0603_1608Metric")
     )
     (path "/b116da63-5dc1-4e35-85cd-0d90c43638cc"
-      (reference "C3") (unit 1) (value "0.1uF") (footprint "Capacitor_SMD:C_0603_1608Metric_Pad1.08x0.95mm_HandSolder")
+      (reference "C3") (unit 1) (value "0.1uF") (footprint "Capacitor_SMD:C_0603_1608Metric")
     )
     (path "/ff325f73-602b-43f6-a40f-7125a406a52a"
-      (reference "C4") (unit 1) (value "0.1uF") (footprint "Capacitor_SMD:C_0603_1608Metric_Pad1.08x0.95mm_HandSolder")
+      (reference "C4") (unit 1) (value "0.1uF") (footprint "Capacitor_SMD:C_0603_1608Metric")
     )
     (path "/21796fa0-b989-4f3e-be7c-54f57fc5be20"
-      (reference "C5") (unit 1) (value "0.1uF") (footprint "Capacitor_SMD:C_0603_1608Metric_Pad1.08x0.95mm_HandSolder")
+      (reference "C5") (unit 1) (value "0.1uF") (footprint "Capacitor_SMD:C_0603_1608Metric")
     )
     (path "/ef48f5dc-9617-4bca-a36a-c2ec7fc594cd"
@@
     )
     (path "/df853e6e-71c4-4a34-83a5-3cde9fd3db09"
-      (reference "J4") (unit 1) (value "Conn_01x08") (footprint "Connector_PinHeader_2.00mm:PinHeader_2x04_P2.00mm_Vertical")
+      (reference "J4") (unit 1) (value "Conn_01x08") (footprint "Connector_PinSocket_2.00mm:PinSocket_2x04_P2.00mm_Vertical_SMD")
     )
     (path "/185a0fb0-4f5c-40c8-b02c-9eda3943ea00"
@@
     )
     (path "/529eedba-99a1-41b2-be43-1ac7449b3764"
-      (reference "R1") (unit 1) (value "10k") (footprint "Resistor_SMD:R_0603_1608Metric_Pad0.98x0.95mm_HandSolder")
+      (reference "R1") (unit 1) (value "10k") (footprint "Resistor_SMD:R_0603_1608Metric")
     )
     (path "/0c2db8df-38d3-47e9-825d-436035963b10"
-      (reference "R2") (unit 1) (value "10k") (footprint "Resistor_SMD:R_0603_1608Metric_Pad0.98x0.95mm_HandSolder")
+      (reference "R2") (unit 1) (value "10k") (footprint "Resistor_SMD:R_0603_1608Metric")
     )
     (path "/ee8bf303-e9bc-49f4-b170-2e808751ac6e"
-      (reference "R3") (unit 1) (value "10k") (footprint "Resistor_SMD:R_0603_1608Metric_Pad0.98x0.95mm_HandSolder")
+      (reference "R3") (unit 1) (value "10k") (footprint "Resistor_SMD:R_0603_1608Metric")
     )
     (path "/7b3bead9-41f1-42b5-ae8f-f77c1ad7da29"
-      (reference "R4") (unit 1) (value "4.7k") (footprint "Resistor_SMD:R_0603_1608Metric_Pad0.98x0.95mm_HandSolder")
+      (reference "R4") (unit 1) (value "4.7k") (footprint "Resistor_SMD:R_0603_1608Metric")
     )
     (path "/61f6679e-4aeb-48f7-94be-933a02f58361"
-      (reference "R5") (unit 1) (value "4.7k") (footprint "Resistor_SMD:R_0603_1608Metric_Pad0.98x0.95mm_HandSolder")
+      (reference "R5") (unit 1) (value "4.7k") (footprint "Resistor_SMD:R_0603_1608Metric")
     )
     (path "/fb2d8904-16bc-479f-905e-94b56ec79c4d"

Commit message: as built PCB rev 1.0
Parts:
- added D1, D2: LED, LED_SMD:LED_0603_1608Metric_Pad1.05x0.95mm_HandSolder, symbol Device:LED
- added H1, H2, H3, H4: MountingHole, MountingHole:MountingHole_2.2mm_M2, symbol Mechanical:MountingHole
- added R6, R7: 330, Resistor_SMD:R_0603_1608Metric, symbol Device:R_US
- C1, C2: CatNo (none) -> 1276-1946-1-ND
- C3, C4, C5: CatNo (none) -> 311-1088-1-ND
- J1, J3: CatNo (none) -> 17-1-2355045-0-ND
- J4: CatNo (none) -> WM23615CT-ND
- R1, R2, R3: CatNo (none) -> RMCF0603FT10K0CT-ND
- R4, R5: CatNo (none) -> RMCF0603FT4K70CT-ND
- U1: CatNo 863-NCP161ASN330T1G -> NCP161ASN330T1GOSCT-ND
Connections:
- net GND: now also D1.1 (K), D2.1 (K)
- net LED1: now reaches U2.7 (XTAL1/PB6)
- net LED1: now also R6.1
- net LED2: now reaches U2.8 (XTAL2/PB7)
- net LED2: now also R7.1
- new net: D1.2 (A), R6.2
- new net: D2.2 (A), R7.2

Commit message: tweak software, schem notes
Connections:
- net SCL: now also U2.28 (PC5); no longer U2.27 (PC4)
- net SDA: now also U2.27 (PC4); no longer U2.28 (PC5)
Other:
- note added: "PCB FIX SDAxSCL"
- note added: "SCL"
- note added: "SDA"
- moved on the sheet: C1, C2, D1, D2, J2, J3, J4, R1, R2, R3, R4, R5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

Commit message: update readme
Parts:
- added Y1: 32.768kHz, symbol Device:Crystal
Connections:
- net at U4.1 (OSCI): now also Y1.1
- net at U4.2 (OSCO): now also Y1.2
Other:
- note added: "Add Y1"
- note added: "Remove I2C pull-ups and use onboard?"
- note added: "Remove R1, R2 or increase?"
Changed lines of the file:
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@@
 		)
 	)
+	(text "Remove I2C pull-ups\nand use onboard?"
+		(exclude_from_sim no)
+		(at 129.794 76.2 0)
+		(effects
+			(font
+				(size 1.27 1.27)
+				(color 255 0 0 1)
+			)
+			(justify left)
+		)
+	)
 	(text "ATMega328 CPU\n\n(should really be e.g. ATMega1281\nbut supply chain...)"
 		(exclude_from_sim no)
@@
 		)
 	)
+	(text "Remove R1, R2\nor increase?"
+		(exclude_from_sim no)
+		(at 24.892 91.44 0)
+		(effects
+			(font
+				(size 1.27 1.27)
+				(color 255 0 0 1)
+			)
+			(justify left)
+		)
+	)
 	(text "UPCO GRAPHICS SYSTEMS"
 		(exclude_from_sim no)
@@
 		)
 	)
+	(text "Add Y1"
+		(exclude_from_sim no)
+		(at 139.954 112.268 0)
+		(effects
+			(font
+				(size 1.27 1.27)
+				(color 255 0 0 1)
+			)
+		)
+	)
 	(text "Battery"
 		(exclude_from_sim no)
@@
 			(font
 				(size 1.27 1.27)
+				(color 255 0 0 1)
 			)
 		)
@@
 	(wire
 		(pts
+			(xy 143.51 110.49) (xy 143.51 100.33)
+		)
+		(stroke
+			(width 0)
+			(type default)
+		)
+	)
+	(wire
+		(pts
 			(xy 83.82 74.93) (xy 83.82 77.47)
 		)
@@
 	(wire
 		(pts
+			(xy 147.32 102.87) (xy 147.32 106.68)
+		)
+		(stroke
+			(width 0)
+			(type default)
+		)
+	)
+	(wire
+		(pts
 			(xy 123.19 161.29) (xy 127 161.29)
 		)
@@
 	(wire
 		(pts
+			(xy 151.13 106.68) (xy 151.13 110.49)
+		)
+		(stroke
+			(width 0)
+			(type default)
+		)
+	)
+	(wire
+		(pts
 			(xy 160.02 128.27) (xy 160.02 134.62)
 		)
@@
 	(wire
 		(pts
+			(xy 143.51 100.33) (xy 147.32 100.33)
+		)
+		(stroke
+			(width 0)
+			(type default)
+		)
+	)
+	(wire
+		(pts
 			(xy 157.48 72.39) (xy 160.02 72.39)
 		)
@@
 	(wire
 		(pts
+			(xy 147.32 106.68) (xy 151.13 106.68)
+		)
+		(stroke
+			(width 0)
+			(type default)
+		)
+	)
+	(wire
+		(pts
 			(xy 29.21 170.18) (xy 35.56 170.18)
 		)
@@
 	)
 	(symbol
+		(lib_id "Device:Crystal")
+		(at 147.32 110.49 0)
+		(unit 1)
+		(exclude_from_sim no)
+		(in_bom yes)
+		(on_board yes)
+		(dnp no)
+		(property "Reference" "Y1"
+			(at 144.526 114.046 0)
+			(effects
+				(font
+					(size 1.27 1.27)
+				)
+			)
+		)
+		(property "Value" "32.768kHz"
+			(at 152.146 114.046 0)
+			(effects
+				(font
+					(size 1.27 1.27)
+				)
+			)
+		)
+		(property "Footprint" ""
+			(at 147.32 110.49 0)
+			(effects
+				(font
+					(size 1.27 1.27)
+				)
+				(hide yes)
+			)
+		)
+		(property "Datasheet" "~"
+			(at 147.32 110.49 0)
+			(effects
+				(font
+					(size 1.27 1.27)
+				)
+				(hide yes)
+			)
+		)
+		(property "Description" "Two pin crystal"
+			(at 147.32 110.49 0)
+			(effects
+				(font
+					(size 1.27 1.27)
+				)
+				(hide yes)
+			)
+		)
+		(pin "1"
+		)
+		(pin "2"
+		)
+		(instances
+			(project ""
+				(path "/970f2a53-dbf3-44e1-b370-568bf247978d"
+					(reference "Y1")
+					(unit 1)
+				)
+			)
+		)
+	)
+	(symbol
 		(lib_id "power:+3.3V")
 		(at 97.79 63.5 0)
@@
 		)
 		(property "Value" "GND"
-			(at 153.67 74.295 0)
+			(at 160.02 74.422 0)
 			(effects
 				(font
